File: jura/jura.sch (EAGLE design)
At the start: 38 parts, among them U1.1 WAGO1255-401-5, U1.2 WAGO1255-401-5, U1.3 WAGO1255-401-5, U1.4 WAGO1255-401-5, U1.5 WAGO1255-401-5, U1.6 WAGO1255-401-5, U1.7 WAGO1255-401-5, U1.8 WAGO1255-401-5

Commit message: more reversing
Parts:
- added C17: (no value), rcl:CPOL-EUE2-4
- added D25, D26: 1N4148DO35-7, diode:1N4148DO35-7
- added L1: (no value), rcl:L-US0204/7
- added R32: (no value), resistor:R-EU_0204/7
- added U6, U7: IL410, optocoupler:IL410
Connections:
- removed net N$13: R35.1, R36.2, ZD2.A
- new net N$17: C17.+, L1.1, U1.8.B1
- new net N$18: R35.1, R36.2, U1.7.B1, ZD2.A
- new net N$19: R25.1, U6.A2
- new net N$20: R27.1, U7.A2
- new net N$21: D26.A, RY41.5, U1.1.B1
- new net N$7: CP2.1.B1, R32.1, RY42.S
- new net N$9: D25.C, L1.2, U1.3.B1
- net GND: now also C17.-, D25.A
- net N$15: now also U6.A1
- net N$16: now also U7.A1
- net N$4: now also R32.2; no longer CP2.1.B1, RY42.S
- net N$5: now also D26.C, RY41.3
Other:
- moved on the sheet: C10, C11, R14, R15, R16, R25, R27, R30, R36, RY4, TM10, TM7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
